Commit message: made minor change to height of kinect (the kinect is still probably too low - also the driver now uses the new description file

File: glados/pharos_description/urdf/pharos1.xacro (robot description, xacro)
@@ -267,5 +267,5 @@
   </link>
   <joint name="base_kinect_joint" type="fixed">
-    <origin xyz="-0.127 0 0.1735" rpy="0 0 0" />
+    <origin xyz="-0.127 0 0.1860" rpy="0 0 0" />
     <parent link="base_link" />
     <child link="kinect_link" />
