Commit message: fixed urdf description with kinect height and added marker, added simple script to test the urdf

File: glados/pharos_description/urdf/pharos1.urdf.xacro (robot description, xacro)
@@ -248,13 +248,13 @@
     </inertial>
   </link>
-  <joint name="laser_joint" type="fixed">
-    <origin xyz="-0.065 0 0.075" rpy="0 0 0" />
+  <joint name="base_marker_joint" type="fixed">
+    <origin xyz="0.093 0 0.123" rpy="0 0 0" />
     <parent link="base_link" />
-    <child link="laser" />
-  </joint>
-  <link name="laser">
-    <visual>
-      <geometry>
-        <box size="0.02 0.035 0.002" />
+    <child link="marker_link" />
+  </joint>
+  <link name="marker_link">
+    <visual>
+      <geometry>
+        <box size="0.228 0.228 0.002" />
       </geometry>
       <material name="Green" />
@@ -269,5 +269,5 @@
   </link>
   <joint name="base_kinect_joint" type="fixed">
-    <origin xyz="-0.127 0 0.1735" rpy="0 0 0" />
+    <origin xyz="-0.127 0 0.233" rpy="0 0 0" />
     <parent link="base_link" />
     <child link="kinect_link" />
