Commit message: re-enabled meshes for collision, mostly to model surface properties properly

File: stacks/bwi/bwi_gazebo/urdf/segbot_base.xacro (robot description, xacro)
@@ -57,5 +57,5 @@
             <origin xyz="0 0 0" rpy="0 0 0" />
             <geometry>
-              <cylinder length="0.56" radius="0.6" />
+              <cylinder length="0.50" radius="0.6" />
               <!-- <mesh filename="package://segbot_description/meshes/rmp50-base-link.dae" scale="0.0254 0.0254 0.0254"/> -->
             </geometry>
@@ -136,12 +136,12 @@
             <origin xyz="0 0 0" rpy="0 0 0" />
             <geometry>
-              <box size="0.01 0.01 0.01" />
-              <!-- <mesh filename="package://segbot_description/meshes/rmp50-castor-wheel.dae" scale="0.0254 0.0254 0.0254"/> -->
+              <!-- <box size="0.01 0.01 0.01" /> -->
+              <mesh filename="package://segbot_description/meshes/rmp50-castor-wheel.dae" scale="0.0254 0.0254 0.0254"/>
             </geometry>
           </collision>
         </link>
         <gazebo reference="caster_wheel_link">
-          <mu1 value="100.0" />
-          <mu2 value="100.0" />
+          <mu1 value="10.0" />
+          <mu2 value="10.0" />
           <kp  value="1000000.0" />
           <kd  value="1.0" />

File: stacks/bwi/bwi_gazebo/urdf/segbot_wheel.xacro (robot description, xacro)
@@ -32,12 +32,12 @@
         <origin xyz="0 0 0" rpy="0 0 0" />
         <geometry>
-          <!-- <mesh filename="package://segbot_description/meshes/rmp50-${suffix}-wheel.dae" scale="0.0254 0.0254 0.0254"/> -->
-          <box size="0.01 0.01 0.01" />
+          <mesh filename="package://segbot_description/meshes/rmp50-${suffix}-wheel.dae" scale="0.0254 0.0254 0.0254"/>
+          <!-- <box size="0.01 0.01 0.01" /> -->
         </geometry>
       </collision>
     </link>
     <gazebo reference="${parent}_${suffix}_wheel_link" >
-      <mu1 value="100.0" />
-      <mu2 value="100.0" />
+      <mu1 value="10.0" />
+      <mu2 value="10.0" />
       <kp  value="1000000.0" />
       <kd  value="1.0" />

Commit message: significant improvements to the real world physics model of the robot, plus works with the new meshes

File: stacks/bwi/bwi_gazebo/urdf/segbot_base.xacro (robot description, xacro)
@@ -34,5 +34,5 @@
         </link>
         <joint name="base_footprint_joint" type="fixed">
-          <origin xyz="0.0 0 0.282" rpy="0 0 0" />
+          <origin xyz="0.0 0 0.2165" rpy="0 0 0" />
           <parent link="base_footprint"/>
           <child link="base_link" />
@@ -43,7 +43,7 @@
             <mass value="5" />
             <origin xyz="0 0 0" />
-            <inertia ixx="0.125" ixy="0.0" ixz="0.0"
-              iyy="0.125" iyz="0.0"
-              izz="0.125" />
+            <inertia ixx="1.0" ixy="0.0" ixz="0.0"
+              iyy="1.0" iyz="0.0"
+              izz="1.0" />
           </inertial>
           <visual>
@@ -57,8 +57,36 @@
             <origin xyz="0 0 0" rpy="0 0 0" />
             <geometry>
-              <cylinder length="0.50" radius="0.6" />
-              <!-- <mesh filename="package://segbot_description/meshes/rmp50-base-link.dae" scale="0.0254 0.0254 0.0254"/> -->
+              <!-- <cylinder length="0.50" radius="0.6" /> -->
+              <mesh filename="package://segbot_description/meshes/rmp50-base-link.dae" scale="0.0254 0.0254 0.0254"/>
             </geometry>
           </collision>
+        </link>
+        <joint name="base_bottom_mass_joint" type="fixed">
+          <origin xyz="0.0 0 -0.15" rpy="0 0 0" />
+          <parent link="base_link"/>
+          <child link="base_bottom_mass_link" />
+        </joint>
+        <link name="base_bottom_mass_link">
+          <inertial>
+            <mass value="15" />
+            <origin xyz="0 0 0" />
+            <inertia ixx="1.0" ixy="0.0" ixz="0.0"
+              iyy="1.0" iyz="0.0"
+              izz="1.0" />
+          </inertial>
+        </link>
+        <joint name="base_rear_mass_joint" type="fixed">
+          <origin xyz="-0.3 0 0" rpy="0 0 0" />
+          <parent link="base_link"/>
+          <child link="base_rear_mass_link" />
+        </joint>
+        <link name="base_rear_mass_link">
+          <inertial>
+            <mass value="10" />
+            <origin xyz="0 0 0" />
+            <inertia ixx="1.0" ixy="0.0" ixz="0.0"
+              iyy="1.0" iyz="0.0"
+              izz="1.0" />
+          </inertial>
         </link>
         <gazebo reference="base_link">
@@ -69,5 +97,5 @@
         </gazebo>
         <joint name="base_caster_support_joint" type="continuous">
-          <origin xyz="-0.2893 0 -0.0185" rpy="0 0 0" />
+          <origin xyz="-0.3292 0 -0.0485" rpy="0 0 0" />
           <parent link="base_link" />
           <child link="base_caster_support_link"/>
@@ -84,5 +112,5 @@
         <link name="base_caster_support_link">
           <inertial>
-            <mass value="2"/>
+            <mass value="1"/>
             <origin xyz="0 0 0" />
             <inertia ixx="0.00375" ixy="0.0" ixz="0.0"
@@ -99,11 +127,11 @@
             <origin xyz="0 0 0" rpy="0 0 0" />
             <geometry>
-              <box size="0.01 0.01 0.01" />
-              <!-- <mesh filename="package://segbot_description/meshes/rmp50-castor-link.dae" scale="0.0254 0.0254 0.0254"/> -->
+              <!-- <box size="0.01 0.01 0.01" /> -->
+              <mesh filename="package://segbot_description/meshes/rmp50-castor-link.dae" scale="0.0254 0.0254 0.0254"/>
             </geometry>
           </collision>
         </link>
         <joint name="caster_wheel_joint" type="continuous">
-          <origin xyz="-0.0382 0 -0.1927" rpy="0 0 0" />
+          <origin xyz="-0.0397 0 -0.0918" rpy="0 0 0" />
           <parent link="base_caster_support_link" />
           <child link="caster_wheel_link" />
@@ -120,13 +148,15 @@
         <link name="caster_wheel_link">
           <inertial>
-            <mass value="0.5" />
-            <origin xyz="0 0 0" rpy="0 0 0" />
-            <inertia  ixx="0.0064" ixy="0.0" ixz="0.0"
-              iyy="0.0122" iyz="0.0"
-              izz="0.0064" />
-          </inertial>
-          <visual>
-            <origin xyz="0 0 0" rpy="0 0 0" />
-            <geometry>
+            <mass value="2" />
+            <origin xyz="0 0 0" rpy="0 0 0" />
+            <inertia  ixx="0.003" ixy="0.0" ixz="0.0"
+              iyy="0.00581" iyz="0.0"
+              izz="0.003" />
+          </inertial>
+          <visual>
+            <origin xyz="0 0 0" rpy="0 0 0" />
+            <!-- <origin xyz="0 0 0" rpy="${M_PI/2} 0 0" /> -->
+            <geometry>
+              <!-- <cylinder radius="0.0762" length="0.0508" /> -->
               <mesh filename="package://segbot_description/meshes/rmp50-castor-wheel.dae" scale="0.0254 0.0254 0.0254"/>
             </geometry>
@@ -135,6 +165,7 @@
           <collision>
             <origin xyz="0 0 0" rpy="0 0 0" />
-            <geometry>
-              <!-- <box size="0.01 0.01 0.01" /> -->
+            <!-- <origin xyz="0 0 0" rpy="${M_PI/2} 0 0" /> -->
+            <geometry>
+              <!-- <cylinder radius="0.0762" length="0.0508" /> -->
               <mesh filename="package://segbot_description/meshes/rmp50-castor-wheel.dae" scale="0.0254 0.0254 0.0254"/>
             </geometry>
@@ -149,8 +180,8 @@
         <!-- MACRO INSTANTIATION -->
         <segbot_wheel suffix="left" parent="base_link">
-          <origin xyz="0 0.2690 -0.0456" rpy="0 0 0" />
+          <origin xyz="0 0.2689 0.0239" rpy="0 0 0" />
         </segbot_wheel>
         <segbot_wheel suffix="right" parent="base_link">
-          <origin xyz="0 -0.2690 -0.0456" rpy="0 0 0" />
+          <origin xyz="0 -0.2689 0.0239" rpy="0 0 0" />
         </segbot_wheel>
         <kinect turtlebot_camera_parent_name="base_link"

File: stacks/bwi/bwi_gazebo/urdf/segbot_wheel.xacro (robot description, xacro)
@@ -18,11 +18,13 @@
         <mass value="5" />
         <origin xyz=" 0 0 0 " />
-        <inertia  ixx="0.633" ixy="0.0" ixz="0.0"
-          iyy="1.26" iyz="0.0"
-          izz="0.633" />
+        <inertia  ixx="0.076" ixy="0.0" ixz="0.0"
+          iyy="0.144" iyz="0.0"
+          izz="0.076" />
       </inertial>
       <visual>
         <origin xyz="0 0 0" rpy="0 0 0" />
+        <!-- <origin xyz="0 0 0" rpy="${M_PI/2} 0 0" /> -->
         <geometry>
+          <!-- <cylinder radius="0.2404" length="0.0952" /> -->
           <mesh filename="package://segbot_description/meshes/rmp50-${suffix}-wheel.dae" scale="0.0254 0.0254 0.0254"/>
         </geometry>
@@ -31,7 +33,8 @@
       <collision>
         <origin xyz="0 0 0" rpy="0 0 0" />
+        <!-- <origin xyz="0 0 0" rpy="${M_PI/2} 0 0" /> -->
         <geometry>
+          <!-- <cylinder radius="0.2404" length="0.0952" /> -->
           <mesh filename="package://segbot_description/meshes/rmp50-${suffix}-wheel.dae" scale="0.0254 0.0254 0.0254"/>
-          <!-- <box size="0.01 0.01 0.01" /> -->
         </geometry>
       </collision>
