Commit message: updated full and simple gazebo models of the robot

File: stacks/pharos_segbot/segbot_description/urdf/gazebo.xacro (robot description, xacro)
@@ -1,4 +1,7 @@
 <?xml version="1.0"?>
-<robot>
+<robot
+  xmlns:sensor="http://playerstage.sourceforge.net/gazebo/xmlschema/#sensor"
+  xmlns:controller="http://playerstage.sourceforge.net/gazebo/xmlschema/#controller"
+  xmlns:interface="http://playerstage.sourceforge.net/gazebo/xmlschema/#interface">
   <!-- Included URDF Files -->
   <include filename="$(find segbot_description)/urdf/gazebo_common.xacro" />
@@ -27,3 +30,9 @@
     <segbot_wheel_mesh suffix="${suffix}" />
   </macro>
+  <macro name="gazebo_segbot_ros_controllers">
+    <gazebo>
+      <gazebo_segbot_drive_plugin />
+      <gazebo_segbot_controllers_common />
+    </gazebo>
+  </macro>
 </robot>

File: stacks/pharos_segbot/segbot_description/urdf/gazebo_common.xacro (robot description, xacro)
@@ -41,5 +41,5 @@
     <origin xyz="0 0 0" rpy="0 0 0" />
     <geometry>
-      <boz size="0.01 0.01 0.01" />
+      <box size="0.01 0.01 0.01" />
     </geometry>
   </macro>
@@ -64,25 +64,33 @@
     </gazebo>
   </macro>
-  <macro name="gazebo_segbot_ros_controllers">
-    <gazebo>
-      <controller:segbotdrive_plugin name="differential_drive_controller" plugin="libsegbotdrive_plugin.so">
-        <alwaysOn>true</alwaysOn>
-        <update>100</update>
-        <updateRate>100.0</updateRate>
-        <leftJoint>base_link_left_wheel_joint</leftJoint>
-        <rightJoint>base_link_right_wheel_joint</rightJoint>
-        <wheelSeparation>0.5380</wheelSeparation>
-        <wheelDiameter>0.2410</wheelDiameter>
-        <torque>20</torque>
-        <interface:position name="position_iface_0"/>
-        <topicName>cmd_vel</topicName>
-      </controller:segbotdrive_plugin>
-      <canonicalBody>base_footprint</canonicalBody>
-      <controller:gazebo_ros_controller_manager name="gazebo_ros_controller_manager" plugin="libgazebo_ros_controller_manager.so">
-        <alwaysOn>true</alwaysOn>
-        <updateRate>5.0</updateRate>
-        <interface:audio name="gazebo_ros_controller_manager_dummy_iface" />
-      </controller:gazebo_ros_controller_manager>
-    </gazebo>
+  <macro name="gazebo_segbot_controllers_common">
+    <canonicalBody>base_footprint</canonicalBody>
+    <controller:gazebo_ros_controller_manager name="gazebo_ros_controller_manager" plugin="libgazebo_ros_controller_manager.so">
+      <alwaysOn>true</alwaysOn>
+      <updateRate>5.0</updateRate>
+      <interface:audio name="gazebo_ros_controller_manager_dummy_iface" />
+    </controller:gazebo_ros_controller_manager>
+  </macro>
+  <macro name="gazebo_segbot_drive_parameters">
+    <alwaysOn>true</alwaysOn>
+    <update>100</update>
+    <updateRate>100.0</updateRate>
+    <leftJoint>base_link_right_wheel_joint</leftJoint>
+    <rightJoint>base_link_left_wheel_joint</rightJoint>
+    <wheelSeparation>0.5380</wheelSeparation>
+    <wheelDiameter>0.2410</wheelDiameter>
+    <torque>20</torque>
+    <interface:position name="position_iface_0"/>
+    <topicName>cmd_vel</topicName>
+  </macro>
+  <macro name="gazebo_segbot_simple_drive_plugin">
+    <controller:segbotsimpledrive_plugin name="differential_drive_controller" plugin="libsegbotsimpledrive_plugin.so">
+      <gazebo_segbot_drive_parameters />
+    </controller:segbotsimpledrive_plugin>
+  </macro>
+  <macro name="gazebo_segbot_drive_plugin">
+    <controller:segbotdrive_plugin name="differential_drive_controller" plugin="libsegbotdrive_plugin.so">
+      <gazebo_segbot_drive_parameters />
+    </controller:segbotdrive_plugin>
   </macro>
 </robot>

File: stacks/pharos_segbot/segbot_description/urdf/segbot_simple.urdf.xacro (robot description, xacro)
@@ -5,5 +5,5 @@
   xmlns:interface="http://playerstage.sourceforge.net/gazebo/xmlschema/#interface">
   <!-- Included URDF Files -->
-  <include filename="$(find segbot_description)/urdf/gazebo.xacro" />
+  <include filename="$(find segbot_description)/urdf/gazebo_simple.xacro" />
   <include filename="$(find segbot_description)/urdf/segbot_base.xacro" />
   <property name="M_PI" value="3.14159"/>
