Commit message: creating simple and complex segbot descriptions -- in process

File: stacks/pharos_segbot/segbot_description/urdf/segbot_base.xacro (robot description, xacro)
@@ -1,7 +1,4 @@
 <?xml version="1.0"?>
-<robot
-  xmlns:sensor="http://playerstage.sourceforge.net/gazebo/xmlschema/#sensor"
-  xmlns:controller="http://playerstage.sourceforge.net/gazebo/xmlschema/#controller"
-  xmlns:interface="http://playerstage.sourceforge.net/gazebo/xmlschema/#interface">
+<robot>
   <!-- Included URDF Files -->
   <include filename="$(find segbot_description)/urdf/segbot_wheel.xacro" />
@@ -15,10 +12,4 @@
         </geometry>
       </visual>
-      <collision>
-        <origin xyz="0 0 0.128" rpy="0 0 0" />
-        <geometry>
-          <box size="0.001 0.001 0.001" />
-        </geometry>
-      </collision>
     </link>
     <joint name="base_footprint_joint" type="fixed">
@@ -30,5 +21,5 @@
     <link name="base_link">
       <inertial>
-        <mass value="5" />
+        <mass value="0.01" />
         <origin xyz="0 0 0" />
         <inertia ixx="1.0" ixy="0.0" ixz="0.0"
@@ -37,25 +28,19 @@
       </inertial>
       <visual>
-        <origin xyz="0 0 0" rpy="0 0 0" />
-        <geometry>
-          <mesh filename="package://segbot_description/meshes/rmp50-base-link.dae" scale="0.0254 0.0254 0.0254"/>
-        </geometry>
+        <segbot_base_link_visual />
       </visual>
       <collision>
-        <origin xyz="0 0 0" rpy="0 0 0" />
-        <geometry>
-          <!-- <cylinder length="0.50" radius="0.6" /> -->
-          <mesh filename="package://segbot_description/meshes/rmp50-base-link.dae" scale="0.0254 0.0254 0.0254"/>
-        </geometry>
+        <segbot_base_link_collision />
       </collision>
     </link>
-    <joint name="base_bottom_mass_joint" type="fixed">
-      <origin xyz="0.0 0 -0.15" rpy="0 0 0" />
+    <gazebo_segbot_base_link_surface />
+    <joint name="base_center_of_mass_joint" type="fixed">
+      <origin xyz="-0.1 0 -0.075" rpy="0 0 0" />
       <parent link="base_link"/>
-      <child link="base_bottom_mass_link" />
+      <child link="base_center_of_mass_link" />
     </joint>
-    <link name="base_bottom_mass_link">
+    <link name="base_center_of_mass_link">
       <inertial>
-        <mass value="15" />
+        <mass value="30" />
         <origin xyz="0 0 0" />
         <inertia ixx="1.0" ixy="0.0" ixz="0.0"
@@ -78,10 +63,4 @@
       </inertial>
     </link>
-    <gazebo reference="base_link">
-      <mu1 value="100.0" />
-      <mu2 value="100.0" />
-      <kp  value="1000000.0" />
-      <kd  value="1.0" />
-    </gazebo>
     <joint name="base_caster_support_joint" type="continuous">
       <origin xyz="-0.3292 0 -0.0485" rpy="0 0 0" />
@@ -107,15 +86,8 @@
       </inertial>
       <visual>
-        <origin xyz="0 0 0" rpy="0 0 0" />
-        <geometry>
-          <mesh filename="package://segbot_description/meshes/rmp50-castor-link.dae" scale="0.0254 0.0254 0.0254"/>
-        </geometry>
+        <segbot_castor_support_link_visual />
       </visual>
       <collision>
-        <origin xyz="0 0 0" rpy="0 0 0" />
-        <geometry>
-          <!-- <box size="0.01 0.01 0.01" /> -->
-          <mesh filename="package://segbot_description/meshes/rmp50-castor-link.dae" scale="0.0254 0.0254 0.0254"/>
-        </geometry>
+        <segbot_castor_support_link_collision />
       </collision>
     </link>
@@ -143,33 +115,20 @@
       </inertial>
       <visual>
-        <origin xyz="0 0 0" rpy="0 0 0" />
-        <!-- <origin xyz="0 0 0" rpy="${M_PI/2} 0 0" /> -->
-        <geometry>
-          <!-- <cylinder radius="0.0762" length="0.0508" /> -->
-          <mesh filename="package://segbot_description/meshes/rmp50-castor-wheel.dae" scale="0.0254 0.0254 0.0254"/>
-        </geometry>
+        <segbot_castor_wheel_link_visual />
       </visual>
       <collision>
-        <origin xyz="0 0 0" rpy="0 0 0" />
-        <!-- <origin xyz="0 0 0" rpy="${M_PI/2} 0 0" /> -->
-        <geometry>
-          <!-- <cylinder radius="0.0762" length="0.0508" /> -->
-          <mesh filename="package://segbot_description/meshes/rmp50-castor-wheel.dae" scale="0.0254 0.0254 0.0254"/>
-        </geometry>
+        <segbot_castor_wheel_link_collision />
       </collision>
     </link>
-    <gazebo reference="caster_wheel_link">
-      <mu1 value="10.0" />
-      <mu2 value="10.0" />
-      <kp  value="1000000.0" />
-      <kd  value="1.0" />
-    </gazebo>
-    <!-- MACRO INSTANTIATION -->
+    <gazebo_castor_wheel_link_surface />
+    <!-- left wheel -->
     <segbot_wheel suffix="left" parent="base_link">
       <origin xyz="0 0.2689 0.0239" rpy="0 0 0" />
     </segbot_wheel>
+    <!-- right wheel -->
     <segbot_wheel suffix="right" parent="base_link">
       <origin xyz="0 -0.2689 0.0239" rpy="0 0 0" />
     </segbot_wheel>
+    <!-- floating kinect (for now) -->
     <kinect turtlebot_camera_parent_name="base_link"
       turtlebot_calib_cam_x="0"
@@ -179,39 +138,6 @@
       turtlebot_calib_cam_rp="0"
       turtlebot_calib_cam_ry="0" />
-    <!-- CONTROLLERS -->
-    <gazebo>
-      <controller:segbotdrive_plugin name="differential_drive_controller" plugin="libsegbotdrive_plugin.so">
-        <alwaysOn>true</alwaysOn>
-        <update>100</update>
-        <updateRate>100.0</updateRate>
-        <leftJoint>base_link_right_wheel_joint</leftJoint>
-        <rightJoint>base_link_left_wheel_joint</rightJoint>
-        <wheelSeparation>0.5380</wheelSeparation>
-        <wheelDiameter>0.2410</wheelDiameter>
-        <torque>20</torque>
-        <interface:position name="position_iface_0"/>
-        <topicName>cmd_vel</topicName>
-      </controller:segbotdrive_plugin>
-      <!-- <controller:gazebo_ros_p3d name="p3d_base_controller" plugin="libgazebo_ros_p3d.so"> -->
-        <!--   <alwaysOn>true</alwaysOn> -->
-        <!--   <updateRate>100.0</updateRate> -->
-        <!--   <bodyName>base_link</bodyName> -->
-        <!--   <topicName>base_pose_ground_truth</topicName> -->
-        <!--   <gaussianNoise>0.01</gaussianNoise> -->
-        <!--   <frameName>map</frameName> -->
-        <!--   <xyzOffsets>0 0 0</xyzOffsets>  -->
-        <!--   <rpyOffsets>0 0 0</rpyOffsets> -->
-        <!--   <interface:position name="p3d_base_position"/> -->
-        <!-- </controller:gazebo_ros_p3d> -->
-      <canonicalBody>base_footprint</canonicalBody>
-      <!-- this publishes empty joint_states due to no transmission, but -->
-      <!--    triggering robot_state_publisher to publish tf between fixed joints in segbot, -->
-      <!--    (e.g. base_laser_link for the base_scan frame) --> -->
-      <controller:gazebo_ros_controller_manager name="gazebo_ros_controller_manager" plugin="libgazebo_ros_controller_manager.so">
-        <alwaysOn>true</alwaysOn>
-        <updateRate>5.0</updateRate>
-        <interface:audio name="gazebo_ros_controller_manager_dummy_iface" />
-      </controller:gazebo_ros_controller_manager>
-    </gazebo>
+    <!-- ros controllers -->
+    <gazebo_segbot_ros_controllers/>
   </macro>
 </robot>

File: stacks/pharos_segbot/segbot_description/urdf/segbot_wheel.xacro (robot description, xacro)
@@ -23,26 +23,11 @@
       </inertial>
       <visual>
-        <origin xyz="0 0 0" rpy="0 0 0" />
-        <!-- <origin xyz="0 0 0" rpy="${M_PI/2} 0 0" /> -->
-        <geometry>
-          <!-- <cylinder radius="0.2404" length="0.0952" /> -->
-          <mesh filename="package://segbot_description/meshes/rmp50-${suffix}-wheel.dae" scale="0.0254 0.0254 0.0254"/>
-        </geometry>
+        <segbot_wheel_visual suffix="${suffix}" />
       </visual>
       <collision>
-        <origin xyz="0 0 0" rpy="0 0 0" />
-        <!-- <origin xyz="0 0 0" rpy="${M_PI/2} 0 0" /> -->
-        <geometry>
-          <!-- <cylinder radius="0.2404" length="0.0952" /> -->
-          <mesh filename="package://segbot_description/meshes/rmp50-${suffix}-wheel.dae" scale="0.0254 0.0254 0.0254"/>
-        </geometry>
+        <segbot_wheel_collision suffix="${suffix}" />
       </collision>
     </link>
-    <gazebo reference="${parent}_${suffix}_wheel_link" >
-      <mu1 value="10.0" />
-      <mu2 value="10.0" />
-      <kp  value="1000000.0" />
-      <kd  value="1.0" />
-    </gazebo>
+    <gazebo_segbot_wheel_surface />
     <transmission type="pr2_mechanism_model/SimpleTransmission" name="${parent}_${suffix}_wheel_trans">
       <actuator name="${parent}_${suffix}_wheel_motor" />

Commit message: removed unnecesary rear mass link in favour of a single center-of-mass link

File: stacks/pharos_segbot/segbot_description/urdf/segbot_base.xacro (robot description, xacro)
@@ -43,18 +43,4 @@
       <inertial>
         <mass value="30" />
-        <origin xyz="0 0 0" />
-        <inertia ixx="1.0" ixy="0.0" ixz="0.0"
-          iyy="1.0" iyz="0.0"
-          izz="1.0" />
-      </inertial>
-    </link>
-    <joint name="base_rear_mass_joint" type="fixed">
-      <origin xyz="-0.3 0 0" rpy="0 0 0" />
-      <parent link="base_link"/>
-      <child link="base_rear_mass_link" />
-    </joint>
-    <link name="base_rear_mass_link">
-      <inertial>
-        <mass value="10" />
         <origin xyz="0 0 0" />
         <inertia ixx="1.0" ixy="0.0" ixz="0.0"
